File: PCB_TrainDriver/H-Bridge_Driver.kicad_sch (KiCad schematic)
At the start: 32 parts, among them J1 Motor1_OUT, J2 Motor2_OUT, Q1 BSC014N04LS, Q2 BSC014N04LS, Q3 BSC014N04LS, Q4 BSC014N04LS, Q5 BSC014N04LS, Q6 BSC014N04LS, Q7 BSC014N04LS, Q8 BSC014N04LS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

Commit message: Update_main_PCB
Parts:
- C11, C14, C5, C6, C7, C8: footprint Capacitor_SMD:CP_Elec_10x7.9 -> Capacitor_SMD:CP_Elec_10x10; JLCPCB Part # (none) -> C46550395
- U1, U2: JLCPCB Part # (none) -> C90964

Commit message: Finished sch
Parts:
- C1, C10, C13, C3, C4, C9: JLCPCB Part # (none) -> C5137482
- C12, C2: JLCPCB Part # (none) -> C49678
- J1, J2: JLCPCB Part # (none) -> C98732
- Q1, Q2, Q3, Q4, Q5, Q6, Q7, Q8: JLCPCB Part # (none) -> C2760081
- R1, R6: JLCPCB Part # (none) -> C4216
- R2, R4: JLCPCB Part # (none) -> C25804
- R3, R5: JLCPCB Part # (none) -> C23231
- U1, U2: LCSC Part Name 有刷直流电机驱动芯片 45V -> (none)

Commit message: PCB Almost Finished
Connections:
- net GH1_1: now also U1.17 (GH1); no longer U1.19 (GL1)
- net GH1_2: now also U2.17 (GH1); no longer U2.19 (GL1)
- net GL1_1: now also U1.19 (GL1); no longer U1.17 (GH1)
- net GL1_2: now also U2.19 (GL1); no longer U2.17 (GH1)
- net SH1_1: now also J1.2 (Pin_2); no longer J1.1 (Pin_1)
- net SH1_2: now also J2.2 (Pin_2); no longer J2.1 (Pin_1)
- net SH2_1: now also J1.1 (Pin_1); no longer J1.2 (Pin_2)
- net SH2_2: now also J2.1 (Pin_1); no longer J2.2 (Pin_2)
