File: PCB_TrainDriver/H-Bridge_Driver.kicad_sch (KiCad schematic)
At the start: 32 parts, among them J1 Motor1_OUT, J2 Motor2_OUT, Q1 BSC014N04LS, Q2 BSC014N04LS, Q3 BSC014N04LS, Q4 BSC014N04LS, Q5 BSC014N04LS, Q6 BSC014N04LS, Q7 BSC014N04LS, Q8 BSC014N04LS, U1 DRV8701ERGER, U2 DRV8701ERGER

Commit message: Finished
Connections:
- net nSLEEP_2 is gone; now on net nSLEEP: U2.13 (nSLEEP)
- net nSLEEP_1 renamed nSLEEP
Changed lines of the file:
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@@
 		)
 	)
-	(hierarchical_label "nSLEEP_2"
+	(hierarchical_label "nSLEEP"
 		(shape input)
 		(at 236.22 78.74 0)
@@
 		)
 	)
-	(hierarchical_label "nSLEEP_1"
+	(hierarchical_label "nSLEEP"
 		(shape input)
 		(at 113.03 78.74 0)
