File: PCB_TrainDriver/MCU.kicad_sch (KiCad schematic)
At the start: 19 parts, among them Q12 SS8050, Q13 SS8050, SW1 SW_Push, U3 ESP32-S3-WROOM-1, U5 CH343P, U7 USBLC6-2P6

Commit message: Finished sch
Parts:
- C15, C16, C17, C18, C29: value 0.1uF -> 0.1uF 50V; JLCPCB Part # (none) -> C307331; LCSC Part # C71687 -> (none)
- C19: value 10uF -> 10uF 10V; JLCPCB Part # (none) -> C2846677; LCSC Part # C77000 -> (none)
- C30: JLCPCB Part # (none) -> C52923; LCSC Part # C14445 -> (none)
- Q12, Q13: JLCPCB Part # (none) -> C2150; LCSC Part # C2150 -> (none)
- R13, R14: JLCPCB Part # (none) -> C23186; LCSC Part # C25905 -> (none)
- R15, R16, R17: JLCPCB Part # (none) -> C25744; LCSC Part # C25744 -> (none)
- SW1: LCSC Part # C318938 -> (none)
- U5: LCSC Part # C2846043 -> (none)
- U7: JLCPCB Part # (none) -> C15999; LCSC Part # C15999 -> (none)
- USB1: JLCPCB Part # (none) -> C393939; LCSC Part # C2765186 -> (none); LCSC Part Name Type-C 母 卧贴 -> (none)
Connections:
- net INA219_SDA: now reaches U3.10 (IO17)
- net INA219_SCL: now reaches U3.11 (IO18)

Commit message: PCB Almost Finished
Parts:
- U5: now fitted
Connections:
- net EN_1: now also U3.6 (IO6); no longer U3.4 (IO4)
- net EN_2: now also U3.18 (IO10); no longer U3.12 (IO8)
- net Horn: now also U3.22 (IO14); no longer U3.21 (IO13)
- net Lamp: now also U3.21 (IO13); no longer U3.22 (IO14)
- net Pneumatic: now also U3.23 (IO21); no longer U3.20 (IO12)
- net nFAULT_1: now also U3.12 (IO8); no longer U3.7 (IO7)
- net nFAULT_2: now also U3.20 (IO12); no longer U3.19 (IO11)
- net nSLEEP_1: now also U3.7 (IO7); no longer U3.6 (IO6)
- net nSLEEP_2: now also U3.19 (IO11); no longer U3.18 (IO10)
- net BackwardIN_3.3V: now reaches U3.16 (IO46)
- net HornIN_3.3V: now reaches U3.24 (IO47)
- net LampIN_3.3V: now reaches U3.25 (IO48)
- net ForwardIN_3.3V: now reaches U3.35 (IO42)
- new net Speed_ControlIN_3.3V: U3.4 (IO4)
- no-connect marks 9 -> 24
Changed lines of the file:
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@@
 	)
 	(no_connect
+		(at 220.98 67.31)
+	)
+	(no_connect
+		(at 251.46 85.09)
+	)
+	(no_connect
 		(at 26.67 36.83)
 	)
 	(no_connect
+		(at 251.46 80.01)
+	)
+	(no_connect
 		(at 53.34 134.62)
 	)
 	(no_connect
+		(at 220.98 62.23)
+	)
+	(no_connect
 		(at 26.67 64.77)
 	)
 	(no_connect
+		(at 220.98 97.79)
+	)
+	(no_connect
 		(at 48.26 59.69)
 	)
 	(no_connect
+		(at 251.46 82.55)
+	)
+	(no_connect
+		(at 251.46 64.77)
+	)
+	(no_connect
 		(at 53.34 132.08)
 	)
 	(no_connect
+		(at 251.46 67.31)
+	)
+	(no_connect
+		(at 251.46 87.63)
+	)
+	(no_connect
+		(at 251.46 77.47)
+	)
+	(no_connect
+		(at 220.98 100.33)
+	)
+	(no_connect
+		(at 251.46 92.71)
+	)
+	(no_connect
+		(at 251.46 74.93)
+	)
+	(no_connect
+		(at 220.98 64.77)
+	)
+	(no_connect
 		(at 53.34 127)
 	)
 	(no_connect
+		(at 251.46 72.39)
+	)
+	(no_connect
 		(at 53.34 129.54)
 	)
@@
 		)
 	)
-	(hierarchical_label "nFAULT_2"
+	(hierarchical_label "ForwardIN_3.3V"
 		(shape input)
-		(at 220.98 87.63 180)
+		(at 251.46 90.17 0)
+		(effects
+			(font
+				(size 1.27 1.27)
+			)
+			(justify left)
+		)
+	)
+	(hierarchical_label "EN_1"
+		(shape output)
+		(at 220.98 74.93 180)
 		(effects
 			(font
@@
 		)
 	)
-	(hierarchical_label "Pneumatic"
+	(hierarchical_label "PH_2"
 		(shape output)
-		(at 220.98 90.17 180)
+		(at 220.98 82.55 180)
+		(effects
+			(font
+				(size 1.27 1.27)
+			)
+			(justify right)
+		)
+	)
+	(hierarchical_label "nFAULT_1"
+		(shape input)
+		(at 220.98 80.01 180)
 		(effects
 			(font
@@
 	(hierarchical_label "nSLEEP_2"
 		(shape output)
-		(at 220.98 85.09 180)
+		(at 220.98 87.63 180)
 		(effects
 			(font
@@
 		)
 	)
-	(hierarchical_label "PH_1"
+	(hierarchical_label "Horn"
 		(shape output)
-		(at 220.98 72.39 180)
+		(at 220.98 95.25 180)
 		(effects
 			(font
@@
 	(hierarchical_label "EN_2"
 		(shape output)
-		(at 220.98 80.01 180)
+		(at 220.98 85.09 180)
 		(effects
 			(font
@@
 		)
 	)
-	(hierarchical_label "nSLEEP_1"
+	(hierarchical_label "BackwardIN_3.3V"
+		(shape input)
+		(at 251.46 95.25 0)
+		(effects
+			(font
+				(size 1.27 1.27)
+			)
+			(justify left)
+		)
+	)
+	(hierarchical_label "Pneumatic"
 		(shape output)
-		(at 220.98 74.93 180)
+		(at 251.46 69.85 0)
 		(effects
 			(font
 				(size 1.27 1.27)
 			)
-			(justify right)
+			(justify left)
 		)
 	)
-	(hierarchical_label "PH_2"
+	(hierarchical_label "Lamp"
 		(shape output)
-		(at 220.98 82.55 180)
+		(at 220.98 92.71 180)
 		(effects
 			(font
@@
 		)
 	)
-	(hierarchical_label "INA219_SDA"
-		(shape bidirectional)
-		(at 251.46 59.69 0)
+	(hierarchical_label "Speed_ControlIN_3.3V"
+		(shape input)
+		(at 220.98 69.85 180)
 		(effects
 			(font
 				(size 1.27 1.27)
 			)
-			(justify left)
+			(justify right)
 		)
 	)
-	(hierarchical_label "EN_1"
+	(hierarchical_label "nSLEEP_1"
 		(shape output)
-		(at 220.98 69.85 180)
+		(at 220.98 77.47 180)
 		(effects
 			(font
@@
 		)
 	)
-	(hierarchical_label "nFAULT_1"
+	(hierarchical_label "LampIN_3.3V"
 		(shape input)
-		(at 220.98 77.47 180)
+		(at 251.46 100.33 0)
 		(effects
 			(font
 				(size 1.27 1.27)
 			)
-			(justify right)
+			(justify left)
 		)
 	)
-	(hierarchical_label "Horn"
-		(shape output)
-		(at 220.98 92.71 180)
+	(hierarchical_label "HornIN_3.3V"
+		(shape input)
+		(at 251.46 97.79 0)
+		(effects
+			(font
+				(size 1.27 1.27)
+			)
+			(justify left)
+		)
+	)
+	(hierarchical_label "nFAULT_2"
+		(shape input)
+		(at 220.98 90.17 180)
 		(effects
 			(font
@@
 		)
 	)
-	(hierarchical_label "Lamp"
+	(hierarchical_label "INA219_SDA"
+		(shape bidirectional)
+		(at 251.46 59.69 0)
+		(effects
+			(font
+				(size 1.27 1.27)
+			)
+			(justify left)
+		)
+	)
+	(hierarchical_label "PH_1"
 		(shape output)
-		(at 220.98 95.25 180)
+		(at 220.98 72.39 180)
 		(effects
 			(font
@@
 		(on_board yes)
 		(in_pos_files yes)
-		(dnp yes)
+		(dnp no)
 		(fields_autoplaced yes)
 		(property "Reference" "U5"
