File: PCB_TrainDriver/MCU.kicad_sch (KiCad schematic)
At the start: 19 parts, among them Q12 SS8050, Q13 SS8050, SW1 SW_Push, U3 ESP32-S3-WROOM-1, U5 CH343P, U7 USBLC6-2P6

Commit message: Finished
Parts:
- added J8: Motor Driver, Connector_JST:JST_XH_B10B-XH-A_1x10_P2.50mm_Vertical, symbol Connector:Conn_01x10_Socket
- added R45: 10k, Resistor_SMD:R_0402_1005Metric, symbol Device:R
- R13, R14: footprint Resistor_SMD:R_0402_1005Metric -> Resistor_SMD:R_0603_1608Metric
- R15, R16, R17: JLCPCB Part # C25744 -> C60490
Connections:
- net +3.3V: now also J8.1 (Pin_1), R45.2
- net BackwardIN_3.3V: now also U3.26 (IO45); no longer U3.16 (IO46)
- net GND: now also J8.2 (Pin_2)
- net GPIO0: now also R45.1
- net Limit1_3.3V: now reaches U3.15 (IO3)
- net EN_4: now reaches U3.32 (IO39)
- net EN_4: now also J8.8 (Pin_8)
- net PH_4: now reaches U3.33 (IO40)
- net PH_4: now also J8.7 (Pin_7)
- net Limit2_3.3V: now reaches U3.34 (IO41)
- net PH_3: now reaches U3.38 (IO2)
- net PH_3: now also J8.3 (Pin_3)
- net EN_3: now reaches U3.39 (IO1)
- net EN_3: now also J8.4 (Pin_4)
- net nFAULT_4: now reaches U3.8 (IO15)
- net nFAULT_4: now also J8.10 (Pin_10)
- net nFAULT_3: now reaches U3.9 (IO16)
- net nFAULT_3: now also J8.6 (Pin_6)
- net nSLEEP_1 renamed nSLEEP
- net nSLEEP: now also J8.5 (Pin_5), J8.9 (Pin_9)
- net nSLEEP_2 renamed Limit4_3.3V
- new net Limit3_3.3V: U3.16 (IO46)
- no-connect marks 24 -> 15
Other:
- moved on the sheet: C18, C19, C29, SW1
