File: PCB_TrainDriver/PCB_TrainDriver.kicad_sch (KiCad schematic)
At the start: 0 parts

Commit message: Update_main_PCB
Other:
- added sheet MCU (MCU.kicad_sch)
- added sheet PSU (PSU.kicad_sch)
- sheet H-Bridge_Driver ports: added EN_1, EN_2, PH_1, PH_2, nFAULT_1, nFAULT_2, nSLEEP_1, nSLEEP_2; removed none
- sheet aux_port ports: added Horn, Lamp, Pneumatic; removed none

Commit message: Finished sch
Other:
- sheet MCU ports: added INA219_SCL, INA219_SDA; removed none
- sheet PSU ports: added INA219_SCL, INA219_SDA; removed none
Changed lines of the file:
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@@
+	(wire
+		(pts
+			(xy 93.98 68.58) (xy 93.98 78.74)
+		)
+		(stroke
+			(width 0)
+			(type default)
+		)
+	)
 	(wire
 		(pts
@@
 		(pts
 			(xy 158.75 138.43) (xy 176.53 138.43)
+		)
+		(stroke
+			(width 0)
+			(type default)
+		)
+	)
+	(wire
+		(pts
+			(xy 97.79 68.58) (xy 97.79 78.74)
 		)
 		(stroke
@@
 			)
 		)
+		(pin "INA219_SCL" bidirectional
+			(at 93.98 68.58 270)
+			(effects
+				(font
+					(size 1.27 1.27)
+				)
+				(justify left)
+			)
+		)
+		(pin "INA219_SDA" bidirectional
+			(at 97.79 68.58 270)
+			(effects
+				(font
+					(size 1.27 1.27)
+				)
+				(justify left)
+			)
+		)
 		(instances
 			(project "PCB_TrainDriver"
@@
 			(effects
 				(font
+					(size 1.27 1.27)
+				)
+				(justify right)
+			)
+		)
+		(pin "INA219_SCL" bidirectional
+			(at 93.98 78.74 90)
+			(effects
+				(font
+					(size 1.27 1.27)
+				)
+				(justify right)
+			)
+		)
+		(pin "INA219_SDA" bidirectional
+			(at 97.79 78.74 90)
+			(effects
+				(font

Commit message: PCB Almost Finished
Parts:
- added H1, H2, H3, H4, H5: MountingHole, MountingHole:MountingHole_5.3mm_M5_DIN965_Pad, symbol Mechanical:MountingHole
Other:
- added sheet Opto (Opto.kicad_sch)
- sheet MCU ports: added BackwardIN_3.3V, ForwardIN_3.3V, HornIN_3.3V, LampIN_3.3V, Speed_ControlIN_3.3V; removed none
