File: PCB_TrainDriver/PCB_TrainDriver.kicad_sch (KiCad schematic)
At the start: 5 parts

Commit message: Finished
Parts:
- added J7: FAN, Connector_JST:JST_XA_B02B-XASK-1_1x02_P2.50mm_Vertical, symbol Connector:Conn_01x02_Pin
Connections:
- new net +12V: J7.2 (Pin_2)
- new net GND: J7.1 (Pin_1)
Other:
- sheet H-Bridge_Driver ports: added nSLEEP; removed nSLEEP_1, nSLEEP_2
- sheet MCU ports: added Limit1_3.3V, Limit2_3.3V, Limit3_3.3V, Limit4_3.3V, nSLEEP; removed nSLEEP_1, nSLEEP_2
- sheet Opto ports: added Limit1_3.3V, Limit2_3.3V, Limit3_3.3V, Limit4_3.3V; removed none
- note added: "Checked"
