File: PCB_TrainDriver/Opto.kicad_sch (KiCad schematic)
At the start: 17 parts, among them J6 JoyStickConnector, U8 TLP291-4

Commit message: Finished
Parts:
- added D14, D15, D16, D17: LED, LED_SMD:LED_0603_1608Metric, symbol Device:LED
- added J10: LimitSW3, Connector_JST:JST_XH_B2B-XH-A_1x02_P2.50mm_Vertical, symbol Connector:Conn_01x02_Socket
- added J11: LimitSW4, Connector_JST:JST_XH_B2B-XH-A_1x02_P2.50mm_Vertical, symbol Connector:Conn_01x02_Socket
- added J12: LimitSW1, Connector_JST:JST_XH_B2B-XH-A_1x02_P2.50mm_Vertical, symbol Connector:Conn_01x02_Socket
- added J9: LimitSW2, Connector_JST:JST_XH_B2B-XH-A_1x02_P2.50mm_Vertical, symbol Connector:Conn_01x02_Socket
- added R37, R39, R40, R43: 22k, Resistor_SMD:R_1206_3216Metric, symbol Device:R_Small
- added R38, R41, R42, R44: 10k, Resistor_SMD:R_0603_1608Metric, symbol Device:R_Small
- added U10: TLP291-4, Package_SO:SOIC-16_4.55x10.3mm_P1.27mm, symbol Isolator:TLP291-4
- J6: JLCPCB Part # (none) -> C144398
- R19: JLCPCB Part # C130232 -> C4216
- R20, R21, R22, R29: JLCPCB Part # C130232 -> C25804
- R28: JLCPCB Part # C22809 -> C25804
- U8: JLCPCB Part # (none) -> C60900
Connections:
- net +12V: now also J10.2 (Pin_2), J11.2 (Pin_2), J12.2 (Pin_2), J9.2 (Pin_2)
- net +3.3V: now also U10.10, U10.12, U10.14, U10.16
- net GND: now also R38.2, R41.2, R42.2, R44.2, U10.2, U10.4, U10.6, U10.8
- new net: D16.1 (K), U10.5
- new net: D16.2 (A), R40.2
- new net: D14.1 (K), U10.1
- new net: D14.2 (A), R37.2
- new net: D17.1 (K), U10.7
- new net: D17.2 (A), R43.2
- new net: D15.1 (K), U10.3
- new net: D15.2 (A), R39.2
- new net Limit1_12V: J12.1 (Pin_1), R37.1
- new net Limit1_3.3V: R38.1, U10.15
- new net Limit2_12V: J9.1 (Pin_1), R39.1
- new net Limit2_3.3V: R41.1, U10.13
- new net Limit3_12V: J10.1 (Pin_1), R40.1
- new net Limit3_3.3V: R42.1, U10.11
- new net Limit4_12V: J11.1 (Pin_1), R43.1
- new net Limit4_3.3V: R44.1, U10.9
Other:
- moved on the sheet: D10, D11, D12, D4, D9, J6, R19, R20, R21, R22, R28, R29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
