File: PCB_TrainDriver/PCB_TrainDriver.kicad_pcb (KiCad board)
At the start: 4 copper layers, 208.5 x 102.3 mm, 136 parts, among them CN1 XT90PW-M.G.Y, J1 Motor1_OUT, J2 Motor2_OUT, J3 aux_port1, J4 aux_port2, J5 aux_port3, J6 JoyStickConnector, Q1 BSC014N04LS, Q10 BSC014N04LS, Q11 BSC014N04LS, Q12 SS8050, Q13 SS8050, Q2 BSC014N04LS, Q3 BSC014N04LS, Q4 BSC014N04LS, Q5 BSC014N04LS, Q6 BSC014N04LS, Q7 BSC014N04LS, Q8 BSC014N04LS, Q9 BSC014N04LS, SW1 SW_Push, U1 DRV8701ERGER, U2 DRV8701ERGER, U3 ESP32-S3-WROOM-1, U4 TPS62932, U5 CH343P, U6 INA219AxDCN, U7 USBLC6-2P6, U8 TLP291-4, U9 LDL1117S33R

Commit message: Finished
Parts:
- added D14: LED, LED_SMD:LED_0603_1608Metric, F.Cu at (159.0, 68.4)
- added D15: LED, LED_SMD:LED_0603_1608Metric, F.Cu at (168.2, 68.0)
- added D16: LED, LED_SMD:LED_0603_1608Metric, F.Cu at (177.6, 68.2)
- added D17: LED, LED_SMD:LED_0603_1608Metric, F.Cu at (187.0, 68.0)
- added J10: LimitSW3, Connector_JST:JST_XH_B2B-XH-A_1x02_P2.50mm_Vertical, F.Cu at (175.4, 75.2)
- added J11: LimitSW4, Connector_JST:JST_XH_B2B-XH-A_1x02_P2.50mm_Vertical, F.Cu at (184.7, 75.1)
- added J12: LimitSW1, Connector_JST:JST_XH_B2B-XH-A_1x02_P2.50mm_Vertical, F.Cu at (156.7, 75.1)
- added J7: FAN, Connector_JST:JST_XA_B02B-XASK-1_1x02_P2.50mm_Vertical, F.Cu at (102.6, 77.5)
- added J8: Motor Driver, Connector_JST:JST_XH_B10B-XH-A_1x10_P2.50mm_Vertical, F.Cu at (72.0, 45.9)
- added J9: LimitSW2, Connector_JST:JST_XH_B2B-XH-A_1x02_P2.50mm_Vertical, F.Cu at (166.0, 75.2)
- added R37: 22k, Resistor_SMD:R_1206_3216Metric, F.Cu at (156.8, 68.6)
- added R38: 10k, Resistor_SMD:R_0603_1608Metric, F.Cu at (179.0, 51.4)
- added R39: 22k, Resistor_SMD:R_1206_3216Metric, F.Cu at (166.0, 68.8)
- added R40: 22k, Resistor_SMD:R_1206_3216Metric, F.Cu at (175.4, 69.0)
- added R41: 10k, Resistor_SMD:R_0603_1608Metric, F.Cu at (181.6, 51.4)
- added R42: 10k, Resistor_SMD:R_0603_1608Metric, F.Cu at (184.2, 51.4)
- added R43: 22k, Resistor_SMD:R_1206_3216Metric, F.Cu at (184.8, 68.8)
- added R44: 10k, Resistor_SMD:R_0603_1608Metric, F.Cu at (186.6, 51.4)
- added R45: 10k, Resistor_SMD:R_0402_1005Metric, F.Cu at (141.8, 70.0)
- added U10: TLP291-4, Package_SO:SOIC-16_4.55x10.3mm_P1.27mm, F.Cu at (182.2, 57.4)
- added kibuzzard-6A50A23A: G***, kibuzzard-6A50A23A, F.Cu at (78.2, 51.8)
- added kibuzzard-6A536EEE: G***, kibuzzard-6A536EEE, F.Cu at (109.0, 78.8)
- added kibuzzard-6A538FDD: G***, kibuzzard-6A538FDD, F.Cu at (155.4, 79.6)
- added kibuzzard-6A538FF4: G***, kibuzzard-6A538FF4, F.Cu at (164.8, 79.6)
- added kibuzzard-6A538FFC: G***, kibuzzard-6A538FFC, F.Cu at (174.2, 79.6)
- added kibuzzard-6A539003: G***, kibuzzard-6A539003, F.Cu at (183.6, 79.6)
- R13, R14: footprint Resistor_SMD:R_0402_1005Metric -> Resistor_SMD:R_0603_1608Metric
- moved kibuzzard-6A412EE2 21.2 mm to (154.8, 44.4), turned to 0 degrees
- moved kibuzzard-6A412F0B 12.8 mm to (154.0, 86.6)
- moved R29 4.60 mm to (201.1, 72.3)
- moved D10 4.60 mm to (204.9, 57.8)
- moved D11 4.60 mm to (207.4, 57.8)
- moved D12 4.60 mm to (209.9, 57.8)
- moved D4 4.60 mm to (196.6, 55.1)
- moved D9 4.60 mm to (202.3, 57.8)
- moved J6 4.60 mm to (199.9, 45.3)
- moved R19 4.60 mm to (199.1, 52.2)
- moved R20 4.60 mm to (208.7, 72.5)
- moved R21 4.60 mm to (206.2, 72.4)
- moved R22 4.60 mm to (203.7, 72.3)
- moved R28 4.60 mm to (195.8, 52.2)
- moved R30 4.60 mm to (202.3, 53.7)
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Connections:
- R34 pad 1: Net-(Q11-G) -> /MCU/Lamp
- R35 pad 1: Net-(Q10-G) -> /MCU/Horn
- R36 pad 1: Net-(Q9-G) -> /MCU/Pneumatic
- U1 pad 13: /H-Bridge_Driver/nSLEEP_1 -> /H-Bridge_Driver/nSLEEP
- U2 pad 13: /H-Bridge_Driver/nSLEEP_2 -> /H-Bridge_Driver/nSLEEP
- U3 pad 15: unconnected-(U3-IO3-Pad15) -> /MCU/Limit1_3.3V
- U3 pad 16: /MCU/BackwardIN_3.3V -> /MCU/Limit3_3.3V
- U3 pad 19: /H-Bridge_Driver/nSLEEP_2 -> /MCU/Limit4_3.3V
- U3 pad 26: unconnected-(U3-IO45-Pad26) -> /MCU/BackwardIN_3.3V
- U3 pad 32: unconnected-(U3-IO39-Pad32) -> /MCU/EN_4
- U3 pad 33: unconnected-(U3-IO40-Pad33) -> /MCU/PH_4
- U3 pad 34: unconnected-(U3-IO41-Pad34) -> /MCU/Limit2_3.3V
- U3 pad 38: unconnected-(U3-IO2-Pad38) -> /MCU/PH_3
- U3 pad 39: unconnected-(U3-IO1-Pad39) -> /MCU/EN_3
- U3 pad 7: /H-Bridge_Driver/nSLEEP_1 -> /H-Bridge_Driver/nSLEEP
- U3 pad 8: unconnected-(U3-IO15-Pad8) -> /MCU/nFAULT_4
- U3 pad 9: unconnected-(U3-IO16-Pad9) -> /MCU/nFAULT_3
Routing:
- net /H-Bridge_Driver/nSLEEP: track 0.00 -> 208.6 mm, vias 0 -> 4
- net /MCU/Limit4_3.3V: track 0.00 -> 98.2 mm, vias 0 -> 2
- net /H-Bridge_Driver/nSLEEP_2: track 91.1 -> 0.00 mm
- net +12V: track 58.1 -> 148.4 mm
- net /MCU/PH_4: track 0.00 -> 82.2 mm, vias 0 -> 2
- net /MCU/EN_4: track 0.00 -> 76.7 mm, vias 0 -> 2
- net /MCU/Limit3_3.3V: track 0.00 -> 66.9 mm, vias 0 -> 2
- net /MCU/PH_3: track 0.00 -> 66.7 mm, vias 0 -> 1
- net /MCU/EN_3: track 0.00 -> 64.3 mm, vias 0 -> 1
- net /MCU/Limit1_3.3V: track 0.00 -> 62.7 mm, vias 0 -> 2
- net /H-Bridge_Driver/nSLEEP_1: track 58.7 -> 0.00 mm
- net /MCU/Limit2_3.3V: track 0.00 -> 57.4 mm
- net /MCU/nFAULT_3: track 0.00 -> 46.3 mm, vias 0 -> 2
- net /MCU/nFAULT_4: track 0.00 -> 38.8 mm, vias 0 -> 2
- net Net-(D14-K): track 0.00 -> 22.6 mm
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