File: PCB_TrainDriver/PSU.kicad_sch (KiCad schematic)
At the start: 27 parts, among them CN1 XT90PW-M.G.Y, U4 TPS62932, U6 INA219AxDCN, U9 LDL1117S33R

Commit message: Finished
Parts:
- R24: JLCPCB Part # C25744 -> C60490
- R27: JLCPCB Part # C25900 -> C11702
Other:
- note added: "Checked"
Changed lines of the file:
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@@
 	(generator_version "10.0")
 	(paper "A4")
+	(text "Checked"
+		(exclude_from_sim no)
+		(at 62.484 116.078 0)
+		(effects
+			(font
+				(face "KiCad Font")
+				(size 1.27 1.27)
+				(thickness 0.254)
+				(bold yes)
+				(color 255 63 23 1)
+			)
+		)
+	)
+	(text "Checked"
+		(exclude_from_sim no)
+		(at 119.126 151.892 0)
+		(effects
+			(font
+				(face "KiCad Font")
+				(size 1.27 1.27)
+				(thickness 0.254)
+				(bold yes)
+				(color 255 63 23 1)
+			)
+		)
+	)
+	(text "Checked"
+		(exclude_from_sim no)
+		(at 139.192 109.22 0)
+		(effects
+			(font
+				(face "KiCad Font")
+				(size 1.27 1.27)
+				(thickness 0.254)
+				(bold yes)
+				(color 255 63 23 1)
+			)
+		)
+	)
 	(junction
 		(at 189.23 111.76)
@@
 			)
 		)
-		(property "JLCPCB Part #" "C25900"
+		(property "JLCPCB Part #" "C11702"
 			(at 218.44 142.24 0)
 			(hide yes)
@@
 			)
 		)
-		(property "JLCPCB Part #" "C25744"
+		(property "JLCPCB Part #" "C60490"
 			(at 189.23 105.41 0)
 			(hide yes)
