File: PCB_TrainDriver/aux_port.kicad_sch (KiCad schematic)
At the start: 21 parts, among them J3 aux_port1, J4 aux_port2, J5 aux_port3, Q10 BSC014N04LS, Q11 BSC014N04LS, Q9 BSC014N04LS

Commit message: Finished
Parts:
- R34, R35, R36: JLCPCB Part # C25900 -> C11702
Connections:
- net Horn: now also R35.1
- net Lamp: now also R34.1
- net Pneumatic: now also R36.1
- net at Q10.4 (G), R10.1, R9.2: no longer R35.1
- net at Q11.4 (G), R11.2, R12.1: no longer R34.1
- net at Q9.4 (G), R7.1, R8.2: no longer R36.1
Other:
- note added: "Checked"
- moved on the sheet: R11, R8, R9
