File: PCB_TrainController/MCU.kicad_sch (KiCad schematic)
At the start: 19 parts, among them Q12 SS8050, Q13 SS8050, SW1 SW_Push, U3 ESP32-S3-WROOM-1, U5 CH343P, U7 USBLC6-2P6

Commit message: Finished
Parts:
- removed USB1: USB-C 16 Pins, Sharing_Footprint:USB-C-SMD_TYPE-C-16PIN, symbol Sharing_Symbol:TYPE-C 16PIN 2MD(073)
- added USB2: (no value), Trainfootprint:USB-C-SMD_TYPE-C-16PIN-2MD-073, symbol TrainDriver:TYPE-C 16PIN 2MD(073)
Connections:
- net +VBUS: now also USB2.A4B9 (VBUS), USB2.B4A9 (VBUS)
- net GND: now also USB2.A1B12 (GND), USB2.B1A12 (GND)
- net at U7.1 (I/O1): now also USB2.A7 (Dn1), USB2.B7 (Dn2)
- net at U7.3 (I/O2): now also USB2.A6 (Dp1), USB2.B6 (Dp2)
- net at R14.1: now also USB2.B5 (CC2)
- net at R13.1: now also USB2.A5 (CC1)
