File: PCB_TrainController/PCB_TrainController.kicad_pcb (KiCad board)
At the start: 4 copper layers, 82 parts, among them J3 aux_port1, J4 aux_port2, J5 aux_port3, J6 JoyStickConnector, J7 Conn_01x10_Socket, Q10 BSC014N04LS, Q11 BSC014N04LS, Q12 SS8050, Q13 SS8050, Q9 BSC014N04LS, SW1 SW_Push, U3 ESP32-S3-WROOM-1, U4 TPS62932, U5 CH343P, U7 USBLC6-2P6, U8 TLP291-4, U9 LDL1117S33R

Commit message: Finished
Parts:
- removed C15, C16, C17, C18, C25, C28, C29: 0.1uF 50V, Capacitor_SMD:C_0402_1005Metric
- removed C19: 10uF 10V, Capacitor_SMD:C_0402_1005Metric
- removed C20: 10uF 50V, Capacitor_SMD:C_1206_3216Metric
- removed C21: 0.1uF 50V, Capacitor_SMD:C_0603_1608Metric
- removed C22: 33nF 10V, Capacitor_SMD:C_0402_1005Metric
- removed C23: 18pF 25V, Capacitor_SMD:C_0402_1005Metric
- removed C24: 47uF 16V, Capacitor_SMD:C_1206_3216Metric
- removed C26, C30, C31: 1uF, Capacitor_SMD:C_0402_1005Metric
- removed C27: 220uF, Capacitor_SMD:C_1206_3216Metric
- removed D1, D2, D3: SS34, Diode_SMD:D_SMA
- removed D10, D11, D12, D13, D6, D7, D8, D9: LED, LED_SMD:LED_0603_1608Metric
- removed D4: BAT54S, Package_TO_SOT_SMD:SOT-23
- removed J5: aux_port3, Connector_AMASS:AMASS_XT30PW-M_1x02_P2.50mm_Horizontal
- removed J7: Conn_01x10_Socket, Connector_JST:JST_XH_B10B-XH-A_1x10_P2.50mm_Vertical
- removed L1: 10uH 21mOhms, Inductor_SMD:L_12x12mm_H4.5mm
- removed Q10, Q11, Q9: BSC014N04LS, Package_SON:Infineon_PG-TDSON-8_6.15x5.15mm
- removed Q12, Q13: SS8050, Package_TO_SOT_SMD:SOT-23
- removed R10, R12, R20, R21, R22, R28, R29, R7: 10k, Resistor_SMD:R_0603_1608Metric
- removed R11, R8, R9: 330, Resistor_SMD:R_0603_1608Metric
- removed R13, R14: 5.1k, Resistor_SMD:R_0402_1005Metric
- removed R15, R16, R17, R24: 10k, Resistor_SMD:R_0402_1005Metric
- removed R19: 33k, Resistor_SMD:R_0603_1608Metric
- removed R23: 52.3k, Resistor_SMD:R_0603_1608Metric
- removed R27, R34, R35, R36: 1k, Resistor_SMD:R_0402_1005Metric
- removed R30, R31, R32, R33: 22k, Resistor_SMD:R_1206_3216Metric
- removed SW1: SW_Push, Button_Switch_SMD:SW_Tactile_SPST_NO_Straight_CK_PTS636Sx25SMTRLFS
- removed TP1: VCC, Connector_Pin:Pin_D0.7mm_L6.5mm_W1.8mm_FlatFork
- removed TP2: 5V, Connector_Pin:Pin_D0.7mm_L6.5mm_W1.8mm_FlatFork
- removed TP3: +3.3V, Connector_Pin:Pin_D0.7mm_L6.5mm_W1.8mm_FlatFork
- removed TP4: GND, Connector_Pin:Pin_D0.7mm_L6.5mm_W1.8mm_FlatFork
- removed U3: ESP32-S3-WROOM-1, RF_Module:ESP32-S3-WROOM-1
- removed U4: TPS62932, Package_TO_SOT_SMD:SOT-583-8
- removed U5: CH343P, Package_DFN_QFN:WCH_QFN-16-1EP_3x3mm_P0.5mm_EP1.8x1.8mm
- removed U7: USBLC6-2P6, Package_TO_SOT_SMD:SOT-666
- removed U8: TLP291-4, Package_SO:SOIC-16_4.55x10.3mm_P1.27mm
- removed U9: LDL1117S33R, Package_TO_SOT_SMD:SOT-223-3_TabPin2
- added J1: Speed_control, Connector_JST:JST_XH_B3B-XH-A_1x03_P2.50mm_Vertical, F.Cu at (105.0, 92.8)
- added J2: LAMP, Connector_JST:JST_XH_B2B-XH-A_1x02_P2.50mm_Vertical, F.Cu at (87.2, 81.3)
- added R1: 10k, Resistor_SMD:R_0805_2012Metric, F.Cu at (95.0, 81.1)
- added R2: 10k, Resistor_SMD:R_0805_2012Metric, F.Cu at (95.0, 89.7)
- added R3: 10k, Resistor_SMD:R_0805_2012Metric, F.Cu at (89.3, 104.4)
- added R4: 10k, Resistor_SMD:R_0805_2012Metric, F.Cu at (86.6, 104.4)
- added R5: 0, Resistor_THT:R_Axial_DIN0204_L3.6mm_D1.6mm_P5.08mm_Horizontal, F.Cu at (98.3, 83.2)
- added R6: 0, Resistor_THT:R_Axial_DIN0204_L3.6mm_D1.6mm_P5.08mm_Horizontal, F.Cu at (98.3, 90.6)
- H1, H2, H3, H4: footprint MountingHole:MountingHole_5.3mm_M5_DIN965_Pad -> MountingHole:MountingHole_3.2mm_M3_DIN965_Pad_TopBottom
- J3: value aux_port1 -> LAMP; footprint Connector_AMASS:AMASS_XT30PW-M_1x02_P2.50mm_Horizontal -> Connector_JST:JST_XH_B2B-XH-A_1x02_P2.50mm_Vertical
- J4: value aux_port2 -> For/Back Control; footprint Connector_AMASS:AMASS_XT30PW-M_1x02_P2.50mm_Horizontal -> Connector_JST:JST_XH_B3B-XH-A_1x03_P2.50mm_Vertical
- J6: footprint Connector_JST:JST_XH_B7B-XH-A_1x07_P2.50mm_Vertical -> Connector_JST:JST_XH_S7B-XH-A_1x07_P2.50mm_Horizontal
- moved J6 117.6 mm to (74.4, 93.5), turned to -90 degrees
- moved J4 66.6 mm to (86.7, 97.8)
- moved H1 65.7 mm to (107.0, 116.0)
- moved H4 58.4 mm to (70.0, 116.0)
- moved J3 54.3 mm to (87.3, 89.7)
- moved H2 51.8 mm to (70.0, 80.0)
- moved H3 13.6 mm to (107.0, 80.0)
Connections:
- J3 pad 1: Net-(D1-A) -> +12V
- J3 pad 2: +12V -> /HornIN_12V
- J4 pad 1: Net-(D2-A) -> /ForwardIN_12V
- J4 pad 2: +12V -> /BackwardIN_12V
- J6 pad 1: /Opto/Speed_ControlIN_12V -> /Speed_ControlIN_12V
- J6 pad 2: /Opto/LampIN_12V -> /LampIN_12V
- J6 pad 3: /Opto/HornIN_12V -> /HornIN_12V
- J6 pad 4: /Opto/BackwardIN_12V -> /BackwardIN_12V
- J6 pad 5: /Opto/ForwardIN_12V -> /ForwardIN_12V
Routing:
- net GND: track 0.00 -> 83.2 mm
- net +12V: track 0.00 -> 74.2 mm
- net /Speed_ControlIN_12V: track 0.00 -> 52.8 mm
- net /LampIN_12V: track 0.00 -> 37.0 mm
- net /BackwardIN_12V: track 0.00 -> 25.1 mm
- net /HornIN_12V: track 0.00 -> 24.9 mm
- net /ForwardIN_12V: track 0.00 -> 17.9 mm
Other:
- board outline added: 45 x 44 mm
- copper layers 4 -> 2
